File: MCU_Datalogger.kicad_pcb (KiCad board)
At the start: 2 copper layers, 0 parts

Commit message: added edge cuts
Other:
- board outline added: 50.4 x 30 mm
Changed lines of the file:
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@@
 	)
 	(property "project_name" " MCU Datalogger with memory and clock")
+	(gr_rect
+		(start 35.6 61.75)
+		(end 86.05 91.7)
+		(stroke
+			(width 0.05)
+			(type default)
+		)
+		(fill no)
+		(layer "Edge.Cuts")
+	)
 	(embedded_fonts no)
 )

Commit message: added power net class
Other:
- copper layers 2 -> 4
Changed lines of the file:
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@@
 	(paper "A4")
 	(layers
-		(0 "F.Cu" signal)
-		(2 "B.Cu" signal)
+		(0 "F.Cu" mixed)
+		(4 "In1.Cu" mixed)
+		(6 "In2.Cu" mixed)
+		(2 "B.Cu" mixed)
 		(9 "F.Adhes" user "F.Adhesive")
 		(11 "B.Adhes" user "B.Adhesive")
@@
 	)
 	(setup
+		(stackup
+			(layer "F.SilkS"
+				(type "Top Silk Screen")
+			)
+			(layer "F.Paste"
+				(type "Top Solder Paste")
+			)
+			(layer "F.Mask"
+				(type "Top Solder Mask")
+				(thickness 0.01)
+			)
+			(layer "F.Cu"
+				(type "copper")
+				(thickness 0.035)
+			)
+			(layer "dielectric 1"
+				(type "prepreg")
+				(thickness 0.1)
+				(material "FR4")
+				(epsilon_r 4.5)
+				(loss_tangent 0.02)
+			)
+			(layer "In1.Cu"
+				(type "copper")
+				(thickness 0.035)
+			)
+			(layer "dielectric 2"
+				(type "core")
+				(thickness 1.24)
+				(material "FR4")
+				(epsilon_r 4.5)
+				(loss_tangent 0.02)
+			)
+			(layer "In2.Cu"
+				(type "copper")
+				(thickness 0.035)
+			)
+			(layer "dielectric 3"
+				(type "prepreg")
+				(thickness 0.1)
+				(material "FR4")
+				(epsilon_r 4.5)
+				(loss_tangent 0.02)
+			)
+			(layer "B.Cu"
+				(type "copper")
+				(thickness 0.035)
+			)
+			(layer "B.Mask"
+				(type "Bottom Solder Mask")
+				(thickness 0.01)
+			)
+			(layer "B.Paste"
+				(type "Bottom Solder Paste")
+			)
+			(layer "B.SilkS"
+				(type "Bottom Silk Screen")
+			)
+			(copper_finish "None")
+			(dielectric_constraints no)
+		)
 		(pad_to_mask_clearance 0)
 		(allow_soldermask_bridges_in_footprints no)
@@
 		(capping no)
 		(filling no)
+		(zone_defaults)
 		(pcbplotparams
 			(layerselection 0x00000000_00000000_55555555_5755f5ff)

Commit message: şematik tamamalandı
Parts:
- added BT1: Battery, Connector_PinHeader_2.54mm:PinHeader_1x02_P2.54mm_Vertical, F.Cu at (138.8, 71.1)
- added C1: 0.1 uF, Capacitor_SMD:C_0805_2012Metric, F.Cu at (134.3, 70.3)
- added C2: 22 pF, Capacitor_SMD:C_0805_2012Metric, F.Cu at (134.3, 73.3)
- added C3: 22 pF, Capacitor_SMD:C_0805_2012Metric, F.Cu at (134.3, 76.3)
- added C4: 0.1 uF, Capacitor_SMD:C_0805_2012Metric, F.Cu at (134.3, 79.3)
- added C5: 100 nF, Capacitor_SMD:C_0805_2012Metric, F.Cu at (134.3, 82.3)
- added D1: LED, LED_SMD:LED_0805_2012Metric, F.Cu at (138.8, 77.5)
- added D2: D, LED_SMD:LED_0805_2012Metric, F.Cu at (138.8, 80.5)
- added H1: MountingHole, MountingHole:MountingHole_2.1mm, F.Cu at (124.8, 61.2)
- added H2: MountingHole, MountingHole:MountingHole_2.1mm, F.Cu at (124.8, 66.9)
- added H3: MountingHole, MountingHole:MountingHole_2.1mm, F.Cu at (124.8, 72.7)
- added H4: MountingHole, MountingHole:MountingHole_2.1mm, F.Cu at (124.8, 78.4)
- added J1: Conn_01x04_Pin, Connector_PinHeader_2.54mm:PinHeader_1x04_P2.54mm_Vertical, F.Cu at (151.2, 60.6)
- added J2: Conn_01x09_Pin, Connector_PinHeader_2.54mm:PinHeader_1x09_P2.54mm_Vertical, F.Cu at (146.6, 60.6)
- added J3: Conn_01x04_Pin, Connector_PinHeader_2.54mm:PinHeader_1x04_P2.54mm_Vertical, F.Cu at (155.8, 60.6)
- added J4: Conn_02x03_Odd_Even, Connector_PinHeader_2.54mm:PinHeader_2x03_P2.54mm_Vertical, F.Cu at (151.2, 72.8)
- added R1: 10 ΚΩ, Resistor_SMD:R_0805_2012Metric, F.Cu at (129.9, 59.8)
- added R2: 10 ΚΩ, Resistor_SMD:R_0805_2012Metric, F.Cu at (129.9, 62.7)
- added R3: 4.7 ΚΩ, Resistor_SMD:R_0805_2012Metric, F.Cu at (129.9, 65.7)
- added R4: 4.7 ΚΩ, Resistor_SMD:R_0805_2012Metric, F.Cu at (129.9, 68.6)
- added R5: 330 Ω, Resistor_SMD:R_0805_2012Metric, F.Cu at (129.9, 71.6)
- added R6: 10 ΚΩ, Resistor_SMD:R_0805_2012Metric, F.Cu at (129.9, 74.5)
- added R7: 330 Ω, Resistor_SMD:R_0805_2012Metric, F.Cu at (129.9, 77.5)
- added U1: DS1337S+, d1337s:SOIC127P600X175-8N, F.Cu at (173.3, 76.1)
- added U2: 24LC1025, 24LC1025:SOIJ8-M_MC_MCH, F.Cu at (171.4, 52.3)
- added U3: 24LC1025, 24LC1025:SOIJ8-M_MC_MCH, F.Cu at (171.4, 58.9)
- added U4: ATMEGA328P-AU, atmega3288p-au:QFP80P900X900X120-32N, F.Cu at (147.4, 51.1)
- added Y1: 32.768 KHz, Crystal:Crystal_SMD_5032-2Pin_5.0x3.2mm_HandSoldering, F.Cu at (137.2, 60.9)
- added Y2: 16 MHz, Crystal:Crystal_SMD_5032-2Pin_5.0x3.2mm_HandSoldering, F.Cu at (137.2, 66.2)

Commit message: PCB design finished
Parts:
- moved U1 114.5 mm to (59.0, 68.9), turned to 180 degrees
- moved J4 111.1 mm to (40.1, 73.2), turned to 180 degrees
- moved J2 106.2 mm to (44.0, 87.8), turned to 90 degrees
- moved Y2 99.9 mm to (38.2, 79.7), turned to 90 degrees
- moved U3 99.3 mm to (74.8, 81.8), turned to 180 degrees
- moved J1 99.2 mm to (52.1, 63.1), turned to -90 degrees
- moved U2 99.0 mm to (74.8, 73.8), turned to 180 degrees
- moved U4 96.2 mm to (55.2, 78.7)
- moved C3 90.8 mm to (43.7, 83.2), turned to 180 degrees
- moved C2 90.7 mm to (43.8, 80.2)
- moved H4 87.4 mm to (38.0, 88.0)
- moved H1 86.8 mm to (38.0, 63.3)
- moved R3 84.9 mm to (45.0, 67.8)
- moved R4 84.8 mm to (45.0, 71.0)
- moved J3 83.3 mm to (77.2, 87.9), turned to -90 degrees
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Routing:
- net /SDA: track 0.00 -> 62.6 mm, vias 0 -> 3
- net /SCL: track 0.00 -> 58.8 mm, vias 0 -> 3
- net /Vcc: track 0.00 -> 37.0 mm, vias 0 -> 12
- net /SCK: track 0.00 -> 27.2 mm, vias 0 -> 1
- net /MISO: track 0.00 -> 26.2 mm, vias 0 -> 1
- net /RX: track 0.00 -> 25.3 mm, vias 0 -> 2
- net /TX: track 0.00 -> 24.7 mm, vias 0 -> 2
- net /RESET: track 0.00 -> 24.6 mm
- net /MOSI: track 0.00 -> 21.6 mm, vias 0 -> 1
- net GND: track 0.00 -> 21.3 mm, vias 0 -> 13
- net /D2: track 0.00 -> 20.1 mm, vias 0 -> 2
- net /D3: track 0.00 -> 15.5 mm, vias 0 -> 2
- net Net-(U4-PB6): track 0.00 -> 14.9 mm
- net Net-(U1-X1): track 0.00 -> 14.8 mm
- net Net-(U4-PB7): track 0.00 -> 14.8 mm
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- added copper zone on B.Cu, net /Vcc
- added copper zone on In1.Cu, net GND
- added copper zone on In2.Cu, net GND
Other:
- board size 50.4 x 30 mm -> 50.5 x 29.9 mm
