File: MCU_Datalogger.kicad_pcb (KiCad board)
At the start: 4 copper layers, 50.5 x 29.9 mm, 30 parts, among them J1 Conn_01x04_Pin, J2 Conn_01x09_Pin, J3 Conn_01x04_Pin, J4 Conn_02x03_Odd_Even, U1 DS1337S+, U2 24LC1025, U3 24LC1025, U4 ATMEGA328P-AU, Y1 32.768 KHz, Y2 16 MHz

Commit message: Added milat footprint
Parts:
- removed REF**: OSHW-Symbol_8.9x8mm_SilkScreen, Symbol:OSHW-Symbol_8.9x8mm_SilkScreen
- added G***: LOGO, KiCadLibs:Milat_Silkscreen_Footprint, F.Cu at (76.0, 65.7)
